File: PCB_GSE/PCB_GSE.kicad_sch (KiCad schematic)
At the start: 0 parts

Commit message: Début schéma moteurs
Other:
- added sheet Interface (Interface.kicad_sch)
- added sheet STM32 (STM32.kicad_sch)
- added sheet Supply (supply.kicad_sch)
Changed lines of the file:
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@@
 	(generator_version "9.0")
 	(paper "A4")
+	(sheet
+		(at 19.05 19.05)
+		(size 76.2 73.66)
+		(exclude_from_sim no)
+		(in_bom yes)
+		(on_board yes)
+		(dnp no)
+		(fields_autoplaced yes)
+		(stroke
+			(width 0.1524)
+			(type solid)
+		)
+		(fill
+			(color 0 0 0 0.0000)
+		)
+		(property "Sheetname" "Supply"
+			(at 19.05 18.3384 0)
+			(effects
+				(font
+					(size 1.27 1.27)
+				)
+				(justify left bottom)
+			)
+		)
+		(property "Sheetfile" "supply.kicad_sch"
+			(at 19.05 93.2946 0)
+			(effects
+				(font
+					(size 1.27 1.27)
+				)
+				(justify left top)
+			)
+		)
+		(instances
+			(project "PCB_GSE"
+				(path "/fb1e7f9a-1970-407a-9a24-5aea0f0ce853"
+					(page "2")
+				)
+			)
+		)
+	)
+	(sheet
+		(at 198.12 19.05)
+		(size 80.01 73.66)
+		(exclude_from_sim no)
+		(in_bom yes)
+		(on_board yes)
+		(dnp no)
+		(fields_autoplaced yes)
+		(stroke
+			(width 0.1524)
+			(type solid)
+		)
+		(fill
+			(color 0 0 0 0.0000)
+		)
+		(property "Sheetname" "Interface"
+			(at 198.12 18.3384 0)
+			(effects
+				(font
+					(size 1.27 1.27)
+				)
+				(justify left bottom)
+			)
+		)
+		(property "Sheetfile" "Interface.kicad_sch"
+			(at 198.12 93.2946 0)
+			(effects
+				(font
+					(size 1.27 1.27)
+				)
+				(justify left top)
+			)
+		)
+		(instances
+			(project "PCB_GSE"
+				(path "/fb1e7f9a-1970-407a-9a24-5aea0f0ce853"
+					(page "4")
+				)
+			)
+		)
+	)
+	(sheet
+		(at 104.14 19.05)
+		(size 83.82 73.66)
+		(exclude_from_sim no)
+		(in_bom yes)
+		(on_board yes)
+		(dnp no)
+		(fields_autoplaced yes)
+		(stroke
+			(width 0.1524)
+			(type solid)
+		)
+		(fill
+			(color 0 0 0 0.0000)
+		)
+		(property "Sheetname" "STM32"
+			(at 104.14 18.3384 0)
+			(effects
+				(font
+					(size 1.27 1.27)
+				)
+				(justify left bottom)
+			)
+		)
+		(property "Sheetfile" "STM32.kicad_sch"
+			(at 104.14 93.2946 0)
+			(effects
+				(font
+					(size 1.27 1.27)
+				)
+				(justify left top)
+			)
+		)
+		(instances
+			(project "PCB_GSE"
+				(path "/fb1e7f9a-1970-407a-9a24-5aea0f0ce853"
+					(page "3")
+				)
+			)
+		)
+	)
 	(sheet_instances
 		(path "/"
