File: Hardware/PCB_Moteur/_autosave-PCB_moteur.kicad_pcb (KiCad board)
At the start: 2 copper layers, 60 x 113 mm, 191 parts, among them J1 XT30PW-F, J10 Conn_01x02, J11 Conn_01x02, J12 Conn_01x02, J13 Conn_01x02, J14 Conn_01x02, J15 Conn_01x02, J16 Conn_01x06_Pin, J17 Screw_Terminal_01x04, J18 Screw_Terminal_01x04, J19 Screw_Terminal_01x04, J2 Conn_01x06_Pin, J3 Conn_01x03_Socket, J4 Conn_01x03_Socket, J5 Conn_01x03_Socket, J6 Conn_01x03_Socket, J7 Conn_01x02, J8 Conn_01x02, J9 Conn_01x02, Q1 SI5442DU-T1-GE3, Q2 SI5442DU-T1-GE3, Q3 MMBT3904, Q4 SI7617DN-T1-GE3, U1 L6981N33DR, U2 STM32F103CBT6, U3 MCP1802T-5002I/OT, U4 LSF0204PWR, U5 ISOW1044, U6 LM393, U7 INA125UA/2K5, U8 INA125UA/2K5, U9 MAX6612MXK

Commit message: wip: fin des circuits sauf ceux du STM
Parts:
- C10, C11, C12, C13: footprint Capacitor_SMD:C_1210_3225Metric -> Capacitor_SMD:C_0805_2012Metric
- moved C25 78.5 mm to (93.5, 48.5), turned to -90 degrees
- moved C26 75.3 mm to (86.5, 50.5), turned to 90 degrees
- moved C24 73.1 mm to (86.5, 47.0), turned to -90 degrees
- moved J2 71.9 mm to (104.8, 103.0), turned to 90 degrees
- moved R18 65.8 mm to (96.0, 48.5), turned to 90 degrees
- moved C28 62.4 mm to (100.5, 90.5), turned to 180 degrees
- moved R22 60.2 mm to (96.1, 82.5)
- moved D13 60.2 mm to (94.7, 51.5)
- moved C27 57.9 mm to (97.0, 90.5)
- moved R24 57.8 mm to (91.6, 73.5)
- moved R12 57.4 mm to (163.6, 95.5)
- moved R19 56.4 mm to (100.0, 82.5)
- moved R20 50.4 mm to (91.5, 85.5)
- moved R23 50.1 mm to (91.5, 79.5)
- moved C11 49.1 mm to (106.1, 64.3)
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Other:
- board size 60 x 113 mm -> 60 x 106.5 mm
- board text added: "decoup 3.3 CAN"
