File: Hardware/PCB_GSE/Comp_user.kicad_sch (KiCad schematic)
At the start: 0 parts

Commit message: un peux d'avancement (brouillon)
Other:
- sheet TransceiverCAN ports: added 3V3, ISO_CAN_IN, ISO_CAN_RXD, ISO_CAN_TXD; removed none
Changed lines of the file:
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@@
 	(generator_version "9.0")
 	(paper "A4")
+	(wire
+		(pts
+			(xy 119.38 68.58) (xy 125.73 68.58)
+		)
+		(stroke
+			(width 0)
+			(type default)
+		)
+	)
+	(wire
+		(pts
+			(xy 82.55 68.58) (xy 85.09 68.58)
+		)
+		(stroke
+			(width 0)
+			(type default)
+		)
+	)
+	(wire
+		(pts
+			(xy 82.55 76.2) (xy 85.09 76.2)
+		)
+		(stroke
+			(width 0)
+			(type default)
+		)
+	)
+	(wire
+		(pts
+			(xy 82.55 71.12) (xy 85.09 71.12)
+		)
+		(stroke
+			(width 0)
+			(type default)
+		)
+	)
+	(hierarchical_label "3V3"
+		(shape input)
+		(at 125.73 68.58 0)
+		(effects
+			(font
+				(size 1.27 1.27)
+			)
+			(justify left)
+		)
+	)
+	(hierarchical_label "ISO_CAN_IN"
+		(shape input)
+		(at 82.55 76.2 180)
+		(effects
+			(font
+				(size 1.27 1.27)
+			)
+			(justify right)
+		)
+	)
+	(hierarchical_label "ISO_CAN_RXD"
+		(shape output)
+		(at 82.55 71.12 180)
+		(effects
+			(font
+				(size 1.27 1.27)
+			)
+			(justify right)
+		)
+	)
+	(hierarchical_label "ISO_CAN_TXD"
+		(shape input)
+		(at 82.55 68.58 180)
+		(effects
+			(font
+				(size 1.27 1.27)
+			)
+			(justify right)
+		)
+	)
 	(sheet
 		(at 85.09 62.23)
-		(size 50.8 20.32)
+		(size 34.29 20.32)
 		(exclude_from_sim no)
 		(in_bom yes)
@@
 			)
 		)
+		(pin "ISO_CAN_IN" input
+			(at 85.09 76.2 180)
+			(effects
+				(font
+					(size 1.27 1.27)
+				)
+				(justify left)
+			)
+		)
+		(pin "ISO_CAN_RXD" output
+			(at 85.09 71.12 180)
+			(effects
+				(font
+					(size 1.27 1.27)
+				)
+				(justify left)
+			)
+		)
+		(pin "ISO_CAN_TXD" input
+			(at 85.09 68.58 180)
+			(effects
+				(font
+					(size 1.27 1.27)
+				)
+				(justify left)
+			)
+		)
+		(pin "3V3" input
+			(at 119.38 68.58 0)
+			(effects
+				(font
+					(size 1.27 1.27)
+				)
+				(justify right)
+			)
+		)
 		(instances
 			(project "PCB_GSE"
@@
 	)
 	(sheet
-		(at 151.13 62.23)
-		(size 50.8 20.32)
+		(at 85.09 90.17)
+		(size 34.29 20.32)
 		(exclude_from_sim no)
 		(in_bom yes)
@@
 		)
 		(property "Sheetname" "Radio"
-			(at 151.13 61.5184 0)
+			(at 85.09 89.4584 0)
 			(effects
 				(font
@@
 		)
 		(property "Sheetfile" "Radio.kicad_sch"
-			(at 151.13 83.1346 0)
+			(at 85.09 111.0746 0)
 			(effects
 				(font
