File: Hardware/PCB_GSE/PressionN20.kicad_sch (KiCad schematic)
At the start: 0 parts

Commit message: un peux d'avancement (brouillon)
Parts:
- added C44, C49: 100nF, Capacitor_SMD:C_0805_2012Metric, symbol Device:C
- added D5: BAT54S, Package_TO_SOT_SMD:SOT-23, symbol Diode:BAT54S
- added J19: Screw_Terminal_01x04, pcb_moteur:CONN_OSTVN04A150_OST, symbol Connector:Screw_Terminal_01x04
- added R53: 10k, Resistor_SMD:R_0805_2012Metric, symbol Device:R
- added R54: 1k, Resistor_SMD:R_0805_2012Metric, symbol Device:R
- added R58: 1.5k, Resistor_SMD:R_0805_2012Metric, symbol Device:R_Small
- added U7: INA125UA/2K5, pcb_moteur:D16-L, symbol pcb_moteur:INA125UA_2K5
Connections:
- new net: D5.3 (COM), R58.1, U7.10 (VO), U7.11 (SENSE)
- new net: R54.2, U7.8 (RG)
- new net: R54.1, U7.9 (RG)
- new net +3.3VA: D5.2 (K)
- new net GND: C44.2, C49.2, D5.1 (A), J19.2 (Pin_2), R53.2, U7.12 (VREFCOM), U7.3 (V-), U7.5 (IAREF)
- new net P_An: C49.1, R58.2
- new net P_IN+: J19.1 (Pin_1), U7.15 (VREF5), U7.4 (VREFOUT)
- new net P_OUT+: J19.3 (Pin_3), U7.6 (V+IN)
- new net P_OUT-: J19.4 (Pin_4), U7.7 (V-IN)
- new net P_SLEEP: R53.1, U7.2 (*SLEEP)
- new net Vin: C44.1, U7.1 (V+)
- no-connect marks 0 -> 3
Other:
- note added: "Active LOW"
- note added: "Pressure"
- note added: "Pressure full scale output typ. 100mV Estimant 100mV max à alimentation typique 10V: On devrait avoir 50mV max à 5V => 3.3V/50mV = 66 V/V Selon datasheet INA125: G = 4+60kOhms/Rg => Rg = 60k/(66-4) = 967 Rg = 1kOhms"
