File: Hardware/PCB_GSE/Temprature.kicad_sch (KiCad schematic)
At the start: 0 parts

Commit message: un peux d'avancement (brouillon)
Parts:
- added C46: 10nF, Capacitor_SMD:C_0603_1608Metric, symbol Device:C
- added C47: 100nF, Capacitor_SMD:C_0805_2012Metric, symbol Device:C
- added U9: MAX6612MXK, Package_TO_SOT_SMD:SOT-353_SC-70-5, symbol MAX6612MXK:MAX6612MXK
Connections:
- new net 3V3: C47.1, U9.4 (VCC)
- new net GND: C46.2, C47.2, U9.1 (A), U9.2 (GND), U9.5 (B)
- new net Temp_An: C46.1, U9.3 (OUT)
Other:
- note added: "Temperature"
