File: Hardware/PCB_GSE/TransceiverCAN.kicad_sch (KiCad schematic)
At the start: 0 parts

Commit message: un peux d'avancement (brouillon)
Parts:
- added C29, C34: 10uF, Capacitor_SMD:C_0805_2012Metric, symbol Device:C
- added C30, C35: 1uF, Capacitor_SMD:C_0805_2012Metric, symbol Device:C
- added C31, C33, C37: 100nF, Capacitor_SMD:C_0805_2012Metric, symbol Device:C
- added C32, C36: 10nF, Capacitor_SMD:C_0603_1608Metric, symbol Device:C
- added FB3: 120R, Inductor_SMD:L_0805_2012Metric, symbol Device:FerriteBead
- added J15: Conn_01x02, pcb_moteur:CONN_2189890010-SD_02_MOL, symbol Connector_Generic:Conn_01x02
- added R34, R35: 60R, Resistor_SMD:R_0805_2012Metric, symbol Device:R
- added U5: ISOW1044, Package_SO:SOIC-20W_7.5x12.8mm_P1.27mm, symbol Interface_CAN_LIN:ISOW1044
Connections:
- new net: J15.2 (Pin_2), R35.1, U5.18 (CANL)
- new net: C37.1, R34.1, R35.2
- new net: J15.1 (Pin_1), R34.2, U5.19 (CANH)
- new net +5VAiso: C34.1, C35.1, C36.1, FB3.2, U5.12 (VISOOUT)
- new net +5Viso: C33.1, FB3.1, U5.13 (VSIN), U5.20 (VISOIN)
- new net 3V3: C29.1, C30.1, C31.1, C32.1, U5.1 (VIO), U5.9 (VDD)
- new net GND: C29.2, C30.2, C31.2, C32.2, U5.10 (GND1), U5.4 (STB), U5.6 (GNDIO)
- new net GND_iso: C33.2, C34.2, C35.2, C36.2, C37.2, U5.11 (GND2), U5.15 (GISOIN), U5.16 (GISOIN), U5.17 (GISOIN)
- new net ISO_CAN_IN: U5.2 (IN)
- new net ISO_CAN_RXD: U5.3 (TXD)
- new net ISO_CAN_TXD: U5.5 (RXD)
- no-connect marks 0 -> 2
Other:
- note added: "CAN"
- note added: "STB -> GND : Normal mode EN/FLT floating : DC-DC enabled (internal pull-up)"
